File: i5ether_mod/i5ether_mod.kicad_pcb (KiCad board)
At the start: 2 copper layers, 24 parts, among them J1 Conn_02x15_Odd_Even, J2 1-406541-1, J3 1-406541-1

Commit message: update
Parts:
- C10, C9: footprint Capacitor_SMD:C_1812_4532Metric_Pad1.57x3.40mm_HandSolder -> Capacitor_SMD:C_0805_2012Metric_Pad1.18x1.45mm_HandSolder
- C11, C12: footprint Capacitor_SMD:C_1812_4532Metric_Pad1.57x3.40mm_HandSolder -> Capacitor_SMD:C_1206_3216Metric_Pad1.33x1.80mm_HandSolder
- J1: footprint Connector_PinSocket_2.54mm:PinSocket_2x15_P2.54mm_Horizontal -> Connector_PinHeader_2.54mm:PinHeader_2x15_P2.54mm_Horizontal; moved to F.Cu
- moved J3 73.1 mm to (166.2, 146.6)
- moved C1 71.2 mm to (124.2, 125.3)
- moved R4 70.0 mm to (149.8, 125.3)
- moved J2 68.3 mm to (166.2, 120.5)
- moved C2 67.5 mm to (124.2, 128.3)
- moved C11 67.1 mm to (160.7, 104.4)
- moved R1 66.5 mm to (149.6, 134.5)
- moved R3 66.3 mm to (149.6, 128.3)
- moved R2 65.3 mm to (149.6, 131.4)
- moved C3 64.7 mm to (124.2, 131.4)
- moved C4 62.3 mm to (124.2, 134.4)
- moved C9 51.6 mm to (148.2, 108.7)
- moved C7 50.2 mm to (124.1, 143.6)
- moved C5 49.6 mm to (124.2, 137.5)
- moved C6 49.3 mm to (124.2, 140.6)
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Connections:
- net Net-(J1-Pad10) renamed /TD7-
- net Net-(J1-Pad11) renamed /TD5+
- net Net-(J1-Pad12) renamed /TD7+
- net Net-(J1-Pad23) renamed /TD1+
- net Net-(J1-Pad24) renamed /TD3+
- net Net-(J1-Pad25) renamed /TD1-
- net Net-(J1-Pad26) renamed /TD3-
- net Net-(J1-Pad27) renamed /TD2-
- net Net-(J1-Pad28) renamed /TD4-
- net Net-(J1-Pad29) renamed /TD2+
- net Net-(J1-Pad30) renamed /TD4+
- net Net-(J1-Pad5) renamed /TD6+
- net Net-(J1-Pad6) renamed /TD8+
- net Net-(J1-Pad7) renamed /TD6-
- net Net-(J1-Pad8) renamed /TD8-
- net Net-(J1-Pad9) renamed /TD5-
- net Net-(J2-Pad1) renamed /MX1+
- net Net-(J2-Pad2) renamed /MX1-
- net Net-(J2-Pad3) renamed /MX2+
- net Net-(J2-Pad4) renamed /MX3+
- net Net-(J2-Pad5) renamed /MX3-
- net Net-(J2-Pad6) renamed /MX2-
- net Net-(J2-Pad7) renamed /MX4+
- net Net-(J2-Pad8) renamed /MX4-
- net Net-(J3-Pad1) renamed /MX5+
- net Net-(J3-Pad2) renamed /MX5-
- net Net-(J3-Pad3) renamed /MX6+
- net Net-(J3-Pad4) renamed /MX7+
- net Net-(J3-Pad5) renamed /MX7-
- net Net-(J3-Pad6) renamed /MX6-
- net Net-(J3-Pad7) renamed /MX8+
- net Net-(J3-Pad8) renamed /MX8-
Routing:
- net GND: track 0.00 -> 44.4 mm, vias 0 -> 9
- net /TD4+: track 0.00 -> 32.7 mm, vias 0 -> 2
- net /TD4-: track 0.00 -> 32.7 mm, vias 0 -> 2
- net /TD3+: track 0.00 -> 29.6 mm
- net /MX6+: track 0.00 -> 27.0 mm
- net /TD3-: track 0.00 -> 26.7 mm, vias 0 -> 2
- net /MX4+: track 0.00 -> 26.5 mm
- net /MX4-: track 0.00 -> 26.0 mm
- net /MX3-: track 0.00 -> 25.8 mm
- net /MX3+: track 0.00 -> 25.7 mm
- net /MX6-: track 0.00 -> 25.6 mm, vias 0 -> 1
- net /MX5+: track 0.00 -> 25.5 mm
- net /MX5-: track 0.00 -> 25.4 mm
- net /MX2+: track 0.00 -> 25.2 mm
- net /TD2+: track 0.00 -> 24.8 mm, vias 0 -> 2
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Other:
- board outline added: 74 x 74 mm

Commit message: update
Parts:
- C11, C12: footprint Capacitor_SMD:C_1206_3216Metric_Pad1.33x1.80mm_HandSolder -> Capacitor_SMD:C_1812_4532Metric_Pad1.57x3.40mm_HandSolder
- moved C10 52.6 mm to (154.0, 100.6)
- moved C12 44.0 mm to (147.5, 121.4)
- moved J3 36.9 mm to (165.1, 109.7)
- moved C1 36.9 mm to (123.0, 88.4)
- moved C5 36.9 mm to (123.1, 100.6)
- moved C6 36.9 mm to (123.1, 103.7)
- moved C7 36.9 mm to (123.0, 106.7)
- moved C8 36.9 mm to (123.1, 109.8)
- moved J1 36.9 mm to (111.4, 117.9)
- moved R1 36.9 mm to (148.5, 97.6)
- moved R2 36.9 mm to (148.5, 94.5)
- moved R3 36.9 mm to (148.5, 91.5)
- moved R5 36.9 mm to (148.5, 109.8)
- moved R7 36.9 mm to (148.5, 103.7)
- moved R8 36.9 mm to (148.5, 100.6)
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- renumbered L1 to T1
Routing:
- net Net-(C9-Pad2): track 16.2 -> 18.6 mm
- net /TD3+: track 29.6 -> 27.2 mm
- net /TD1+: track 23.6 -> 21.2 mm
- net Net-(C10-Pad2): track 16.4 -> 17.9 mm
- net /TD4+: track 32.7 -> 31.7 mm, vias 2 -> 1
- net /TD4-: track 32.7 -> 31.7 mm, vias 2 -> 1
- net /TD3-: track 26.7 -> 25.7 mm, vias 2 -> 1
- net /TD1-: track 19.8 -> 18.9 mm, vias 2 -> 1
- net /TD2+: track 24.8 -> 25.7 mm, vias 2 -> 1
- net /TD2-: track 24.8 -> 24.2 mm
- added copper zone on B.Cu, net Earth
- added copper zone on F.Cu, net Earth
- added copper zone on B.Cu, net GND
- added copper zone on F.Cu, net GND

Commit message: update
Parts:
- C10, C9: value 1000p -> 1n
- C11, C12: value 4700p -> 4.7n
- renumbered R4 to R1, R3 to R2, R2 to R3, R1 to R4, R8 to R5, R7 to R6, R6 to R7, R5 to R8

Commit message: final
Parts:
- added H1: MountingHole_Pad, MountingHole:MountingHole_3.2mm_M3_Pad, F.Cu at (102.6, 66.8)
- added H2: MountingHole_Pad, MountingHole:MountingHole_3.2mm_M3_Pad, F.Cu at (102.6, 133.4)
- added H3: MountingHole_Pad, MountingHole:MountingHole_3.2mm_M3_Pad, F.Cu at (169.1, 133.4)
- added H4: MountingHole_Pad, MountingHole:MountingHole_3.2mm_M3_Pad, F.Cu at (169.1, 66.9)
- added REF**: KiCad-Logo2_5mm_SilkScreen, Symbol:KiCad-Logo2_5mm_SilkScreen, F.Cu at (115.2, 129.5)
- added REF**: OSHW-Logo2_7.3x6mm_SilkScreen, Symbol:OSHW-Logo2_7.3x6mm_SilkScreen, F.Cu at (127.0, 129.7)
- added REF**: OSHW-Logo2_7.3x6mm_SilkScreen, Symbol:OSHW-Logo2_7.3x6mm_SilkScreen, B.Cu at (126.5, 70.4)
- added REF**: KiCad-Logo2_5mm_SilkScreen, Symbol:KiCad-Logo2_5mm_SilkScreen, B.Cu at (114.7, 70.6)
Routing:
- net GND: track 44.9 -> 34.5 mm, vias 9 -> 65
- net Earth: vias 0 -> 25
Other:
- board text added: "Colorlight I5 Ethernet Adaptor Module"
- board text added: "Rev V1.0"

Commit message: final
Parts:
- C1, C2, C3, C4, C5, C6, C7, C8: value 0.1u -> 100n
