File: i5ether_mod/i5ether_mod.kicad_sch (KiCad schematic)
At the start: 24 parts, among them J1 Conn_02x15_Odd_Even, J2 1-406541-1, J3 1-406541-1, U1 PM6C-2004F

Commit message: update
Parts:
- J1: footprint (none) -> Connector_PinSocket_2.54mm:PinSocket_2x15_P2.54mm_Horizontal
- J2, J3: footprint CONN8_406541_TEC -> MJ406541:1-406541-1
- L1: renamed from U1; footprint (none) -> PM6C-200XF:PM6C-2004F_SOP48
Changed lines of the file:
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@@
       (effects (font (size 1.524 1.524)) (justify left))
     )
-    (property "Footprint" "CONN8_406541_TEC" (id 2) (at 213.36 71.374 0)
+    (property "Footprint" "MJ406541:1-406541-1" (id 2) (at 213.36 71.374 0)
       (effects (font (size 1.524 1.524)) hide)
     )
@@
       (effects (font (size 1.524 1.524)) (justify left))
     )
-    (property "Footprint" "CONN8_406541_TEC" (id 2) (at 213.36 104.394 0)
+    (property "Footprint" "MJ406541:1-406541-1" (id 2) (at 213.36 104.394 0)
       (effects (font (size 1.524 1.524)) hide)
     )
@@
   (symbol (lib_id "PM6C-200XF:PM6C-2004F") (at 143.51 87.63 0) (unit 1)
     (in_bom yes) (on_board yes) (fields_autoplaced)
-    (property "Reference" "U1" (id 0) (at 143.51 52.07 0))
+    (property "Reference" "L1" (id 0) (at 143.51 52.07 0))
     (property "Value" "PM6C-2004F" (id 1) (at 143.51 54.61 0))
-    (property "Footprint" "" (id 2) (at 133.35 111.76 0)
+    (property "Footprint" "PM6C-200XF:PM6C-2004F_SOP48" (id 2) (at 133.35 111.76 0)
       (effects (font (size 1.27 1.27)) hide)
     )
@@
     (property "Reference" "J1" (id 0) (at 88.9 67.31 0))
     (property "Value" "Conn_02x15_Odd_Even" (id 1) (at 88.9 107.95 0))
-    (property "Footprint" "" (id 2) (at 87.63 87.63 0)
+    (property "Footprint" "Connector_PinSocket_2.54mm:PinSocket_2x15_P2.54mm_Horizontal" (id 2) (at 87.63 87.63 0)
       (effects (font (size 1.27 1.27)) hide)
     )
@@
     )
     (path "/efe23ee3-88d7-4a07-85ed-8af6a1b1b716"
-      (reference "J1") (unit 1) (value "Conn_02x15_Odd_Even") (footprint "")
+      (reference "J1") (unit 1) (value "Conn_02x15_Odd_Even") (footprint "Connector_PinSocket_2.54mm:PinSocket_2x15_P2.54mm_Horizontal")
     )
     (path "/31ec8395-3404-4709-afd7-258f2db671a8"
-      (reference "J2") (unit 1) (value "1-406541-1") (footprint "CONN8_406541_TEC")
+      (reference "J2") (unit 1) (value "1-406541-1") (footprint "MJ406541:1-406541-1")
     )
     (path "/5d60c08b-b737-4800-a755-ec72e7fb79d3"
-      (reference "J3") (unit 1) (value "1-406541-1") (footprint "CONN8_406541_TEC")
+      (reference "J3") (unit 1) (value "1-406541-1") (footprint "MJ406541:1-406541-1")
+    )
+    (path "/bfa46546-c392-46f2-9dd1-54c070a9f47d"
+      (reference "L1") (unit 1) (value "PM6C-2004F") (footprint "PM6C-200XF:PM6C-2004F_SOP48")
     )
     (path "/98624091-3add-4002-a75e-32916797ae00"
@@
       (reference "R8") (unit 1) (value "75") (footprint "Resistor_SMD:R_0805_2012Metric_Pad1.20x1.40mm_HandSolder")
     )
-    (path "/bfa46546-c392-46f2-9dd1-54c070a9f47d"
-      (reference "U1") (unit 1) (value "PM6C-2004F") (footprint "")
-    )
-  )
+  )

Commit message: update
Parts:
- C10, C9: footprint Capacitor_SMD:C_1812_4532Metric_Pad1.57x3.40mm_HandSolder -> Capacitor_SMD:C_0805_2012Metric_Pad1.18x1.45mm_HandSolder
- C11, C12: footprint Capacitor_SMD:C_1812_4532Metric_Pad1.57x3.40mm_HandSolder -> Capacitor_SMD:C_1206_3216Metric_Pad1.33x1.80mm_HandSolder
- J1: footprint Connector_PinSocket_2.54mm:PinSocket_2x15_P2.54mm_Horizontal -> Connector_PinHeader_2.54mm:PinHeader_2x15_P2.54mm_Horizontal
Connections:
- net MX1+: now reaches J2.1, L1.47 (MX1+)
- net MX1-: now reaches J2.2, L1.46 (MX1-)
- net MX2+: now reaches J2.3, L1.44 (MX2+)
- net MX3+: now reaches J2.4, L1.41 (MX3+)
- net MX3-: now reaches J2.5, L1.40 (MX3-)
- net MX2-: now reaches J2.6, L1.43 (MX2-)
- net MX4+: now reaches J2.7, L1.38 (MX4+)
- net MX4-: now reaches J2.8, L1.37 (MX4-)
- net MX5+: now reaches J3.1, L1.35 (MX5+)
- net MX5-: now reaches J3.2, L1.34 (MX5-)
- net MX6+: now reaches J3.3, L1.32 (MX6+)
- net MX7+: now reaches J3.4, L1.29 (MX7+)
- net MX7-: now reaches J3.5, L1.28 (MX7-)
- net MX6-: now reaches J3.6, L1.31 (MX6-)
- net MX8+: now reaches J3.7, L1.26 (MX8+)
- net MX8-: now reaches J3.8, L1.25 (MX8-)
- net TD4+: now reaches J1.30 (Pin_30), L1.11 (TD4+)
- net TD4-: now reaches J1.28 (Pin_28), L1.12 (TD4-)
- net TD5+: now reaches J1.11 (Pin_11), L1.14 (TD5+)
- net TD5-: now reaches J1.9 (Pin_9), L1.15 (TD5-)
- net TD6+: now reaches J1.5 (Pin_5), L1.17 (TD6+)
- net TD6-: now reaches J1.7 (Pin_7), L1.18 (TD6-)
- net TD1+: now reaches J1.23 (Pin_23), L1.2 (TD1+)
- net TD7+: now reaches J1.12 (Pin_12), L1.20 (TD7+)
- net TD7-: now reaches J1.10 (Pin_10), L1.21 (TD7-)
- net TD8+: now reaches J1.6 (Pin_6), L1.23 (TD8+)
- net TD8-: now reaches J1.8 (Pin_8), L1.24 (TD8-)
- net TD1-: now reaches J1.25 (Pin_25), L1.3 (TD1-)
- net TD2+: now reaches J1.29 (Pin_29), L1.5 (TD2+)
- net TD2-: now reaches J1.27 (Pin_27), L1.6 (TD2-)
- net TD3+: now reaches J1.24 (Pin_24), L1.8 (TD3+)
- net TD3-: now reaches J1.26 (Pin_26), L1.9 (TD3-)
Changed lines of the file:
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@@
     (stroke (width 0) (type default) (color 0 0 0 0))
+  )
+  (label "MX7+" (at 152.4 106.68 0)
+    (effects (font (size 1.27 1.27)) (justify left bottom))
+  )
+  (label "MX7-" (at 152.4 109.22 0)
+    (effects (font (size 1.27 1.27)) (justify left bottom))
+  )
+  (label "MX8+" (at 152.4 114.3 0)
+    (effects (font (size 1.27 1.27)) (justify left bottom))
+  )
+  (label "MX2-" (at 152.4 71.12 0)
+    (effects (font (size 1.27 1.27)) (justify left bottom))
+  )
+  (label "MX5+" (at 152.4 91.44 0)
+    (effects (font (size 1.27 1.27)) (justify left bottom))
+  )
+  (label "TD5+" (at 118.11 91.44 0)
+    (effects (font (size 1.27 1.27)) (justify left bottom))
+  )
+  (label "MX6-" (at 152.4 101.6 0)
+    (effects (font (size 1.27 1.27)) (justify left bottom))
+  )
+  (label "MX2+" (at 152.4 68.58 0)
+    (effects (font (size 1.27 1.27)) (justify left bottom))
+  )
+  (label "TD5-" (at 118.11 93.98 0)
+    (effects (font (size 1.27 1.27)) (justify left bottom))
+  )
+  (label "TD4-" (at 118.11 86.36 0)
+    (effects (font (size 1.27 1.27)) (justify left bottom))
+  )
+  (label "MX1+" (at 152.4 60.96 0)
+    (effects (font (size 1.27 1.27)) (justify left bottom))
+  )
+  (label "TD7-" (at 118.11 109.22 0)
+    (effects (font (size 1.27 1.27)) (justify left bottom))
+  )
+  (label "TD3-" (at 118.11 78.74 0)
+    (effects (font (size 1.27 1.27)) (justify left bottom))
+  )
+  (label "MX4-" (at 152.4 86.36 0)
+    (effects (font (size 1.27 1.27)) (justify left bottom))
+  )
+  (label "TD4+" (at 118.11 83.82 0)
+    (effects (font (size 1.27 1.27)) (justify left bottom))
+  )
+  (label "MX8-" (at 152.4 116.84 0)
+    (effects (font (size 1.27 1.27)) (justify left bottom))
+  )
+  (label "MX3+" (at 152.4 76.2 0)
+    (effects (font (size 1.27 1.27)) (justify left bottom))
+  )
+  (label "TD7+" (at 118.11 106.68 0)
+    (effects (font (size 1.27 1.27)) (justify left bottom))
+  )
+  (label "MX1-" (at 152.4 63.5 0)
+    (effects (font (size 1.27 1.27)) (justify left bottom))
+  )
+  (label "TD6+" (at 118.11 99.06 0)
+    (effects (font (size 1.27 1.27)) (justify left bottom))
+  )
+  (label "TD1+" (at 118.11 60.96 0)
+    (effects (font (size 1.27 1.27)) (justify left bottom))
+  )
+  (label "TD1-" (at 118.11 63.5 0)
+    (effects (font (size 1.27 1.27)) (justify left bottom))
+  )
+  (label "MX4+" (at 152.4 83.82 0)
+    (effects (font (size 1.27 1.27)) (justify left bottom))
+  )
+  (label "MX5-" (at 152.4 93.98 0)
+    (effects (font (size 1.27 1.27)) (justify left bottom))
+  )
+  (label "MX3-" (at 152.4 78.74 0)
+    (effects (font (size 1.27 1.27)) (justify left bottom))
+  )
+  (label "TD6-" (at 118.11 101.6 0)
+    (effects (font (size 1.27 1.27)) (justify left bottom))
+  )
+  (label "MX6+" (at 152.4 99.06 0)
+    (effects (font (size 1.27 1.27)) (justify left bottom))
+  )
+  (label "TD8-" (at 118.11 116.84 0)
+    (effects (font (size 1.27 1.27)) (justify left bottom))
+  )
+  (label "TD2+" (at 118.11 68.58 0)
+    (effects (font (size 1.27 1.27)) (justify left bottom))
+  )
+  (label "TD2-" (at 118.11 71.12 0)
+    (effects (font (size 1.27 1.27)) (justify left bottom))
+  )
+  (label "TD3+" (at 118.11 76.2 0)
+    (effects (font (size 1.27 1.27)) (justify left bottom))
+  )
+  (label "TD8+" (at 118.11 114.3 0)
+    (effects (font (size 1.27 1.27)) (justify left bottom))
   )
   (symbol (lib_id "Device:C") (at 116.84 133.35 0) (unit 1)
@@
       (effects (font (size 1.27 1.27)) (justify left))
     )
-    (property "Footprint" "Capacitor_SMD:C_1812_4532Metric_Pad1.57x3.40mm_HandSolder" (id 2) (at 144.78 138.1252 0)
+    (property "Footprint" "Capacitor_SMD:C_1206_3216Metric_Pad1.33x1.80mm_HandSolder" (id 2) (at 144.78 138.1252 0)
       (effects (font (size 1.27 1.27)) hide)
     )
@@
       (effects (font (size 1.27 1.27)) (justify left))
     )
-    (property "Footprint" "Capacitor_SMD:C_1812_4532Metric_Pad1.57x3.40mm_HandSolder" (id 2) (at 184.15 119.0752 0)
+    (property "Footprint" "Capacitor_SMD:C_0805_2012Metric_Pad1.18x1.45mm_HandSolder" (id 2) (at 184.15 119.0752 0)
       (effects (font (size 1.27 1.27)) hide)
     )
@@
       (effects (font (size 1.27 1.27)) (justify left))
     )
-    (property "Footprint" "Capacitor_SMD:C_1812_4532Metric_Pad1.57x3.40mm_HandSolder" (id 2) (at 144.78 133.0452 0)
+    (property "Footprint" "Capacitor_SMD:C_1206_3216Metric_Pad1.33x1.80mm_HandSolder" (id 2) (at 144.78 133.0452 0)
       (effects (font (size 1.27 1.27)) hide)
     )
@@
       (effects (font (size 1.27 1.27)) (justify left))
     )
-    (property "Footprint" "Capacitor_SMD:C_1812_4532Metric_Pad1.57x3.40mm_HandSolder" (id 2) (at 184.15 87.3252 0)
+    (property "Footprint" "Capacitor_SMD:C_0805_2012Metric_Pad1.18x1.45mm_HandSolder" (id 2) (at 184.15 87.3252 0)
       (effects (font (size 1.27 1.27)) hide)
     )
@@
     (property "Reference" "J1" (id 0) (at 88.9 67.31 0))
     (property "Value" "Conn_02x15_Odd_Even" (id 1) (at 88.9 107.95 0))
-    (property "Footprint" "Connector_PinSocket_2.54mm:PinSocket_2x15_P2.54mm_Horizontal" (id 2) (at 87.63 87.63 0)
+    (property "Footprint" "Connector_PinHeader_2.54mm:PinHeader_2x15_P2.54mm_Horizontal" (id 2) (at 87.63 87.63 0)
       (effects (font (size 1.27 1.27)) hide)
     )
@@
     )
     (path "/b359cff7-6ac7-45fb-b749-9bcb9a702089"
-      (reference "C9") (unit 1) (value "1000p") (footprint "Capacitor_SMD:C_1812_4532Metric_Pad1.57x3.40mm_HandSolder")
+      (reference "C9") (unit 1) (value "1000p") (footprint "Capacitor_SMD:C_0805_2012Metric_Pad1.18x1.45mm_HandSolder")
     )
     (path "/8b687076-a1d3-4ddc-b349-bb354de157f8"
-      (reference "C10") (unit 1) (value "1000p") (footprint "Capacitor_SMD:C_1812_4532Metric_Pad1.57x3.40mm_HandSolder")
+      (reference "C10") (unit 1) (value "1000p") (footprint "Capacitor_SMD:C_0805_2012Metric_Pad1.18x1.45mm_HandSolder")
     )
     (path "/8fadaaf1-6657-4bb6-bf18-fe2c1d6327ef"
-      (reference "C11") (unit 1) (value "4700p") (footprint "Capacitor_SMD:C_1812_4532Metric_Pad1.57x3.40mm_HandSolder")
+      (reference "C11") (unit 1) (value "4700p") (footprint "Capacitor_SMD:C_1206_3216Metric_Pad1.33x1.80mm_HandSolder")
     )
     (path "/6235df39-6fe4-4ff0-a6f7-da05e5c190f5"
-      (reference "C12") (unit 1) (value "4700p") (footprint "Capacitor_SMD:C_1812_4532Metric_Pad1.57x3.40mm_HandSolder")
+      (reference "C12") (unit 1) (value "4700p") (footprint "Capacitor_SMD:C_1206_3216Metric_Pad1.33x1.80mm_HandSolder")
     )
     (path "/efe23ee3-88d7-4a07-85ed-8af6a1b1b716"
-      (reference "J1") (unit 1) (value "Conn_02x15_Odd_Even") (footprint "Connector_PinSocket_2.54mm:PinSocket_2x15_P2.54mm_Horizontal")
+      (reference "J1") (unit 1) (value "Conn_02x15_Odd_Even") (footprint "Connector_PinHeader_2.54mm:PinHeader_2x15_P2.54mm_Horizontal")
     )
     (path "/31ec8395-3404-4709-afd7-258f2db671a8"

Commit message: update
Parts:
- C11, C12: footprint Capacitor_SMD:C_1206_3216Metric_Pad1.33x1.80mm_HandSolder -> Capacitor_SMD:C_1812_4532Metric_Pad1.57x3.40mm_HandSolder
- renumbered L1 to T1
Changed lines of the file:
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@@
       (effects (font (size 1.27 1.27)) (justify left))
     )
-    (property "Footprint" "Capacitor_SMD:C_1206_3216Metric_Pad1.33x1.80mm_HandSolder" (id 2) (at 144.78 138.1252 0)
+    (property "Footprint" "Capacitor_SMD:C_1812_4532Metric_Pad1.57x3.40mm_HandSolder" (id 2) (at 144.78 138.1252 0)
       (effects (font (size 1.27 1.27)) hide)
     )
@@
       (effects (font (size 1.27 1.27)) (justify left))
     )
-    (property "Footprint" "Capacitor_SMD:C_1206_3216Metric_Pad1.33x1.80mm_HandSolder" (id 2) (at 144.78 133.0452 0)
+    (property "Footprint" "Capacitor_SMD:C_1812_4532Metric_Pad1.57x3.40mm_HandSolder" (id 2) (at 144.78 133.0452 0)
       (effects (font (size 1.27 1.27)) hide)
     )
@@
   (symbol (lib_id "PM6C-200XF:PM6C-2004F") (at 143.51 87.63 0) (unit 1)
     (in_bom yes) (on_board yes) (fields_autoplaced)
-    (property "Reference" "L1" (id 0) (at 143.51 52.07 0))
+    (property "Reference" "T1" (id 0) (at 143.51 52.07 0))
     (property "Value" "PM6C-2004F" (id 1) (at 143.51 54.61 0))
     (property "Footprint" "PM6C-200XF:PM6C-2004F_SOP48" (id 2) (at 133.35 111.76 0)
@@
     )
     (path "/8fadaaf1-6657-4bb6-bf18-fe2c1d6327ef"
-      (reference "C11") (unit 1) (value "4700p") (footprint "Capacitor_SMD:C_1206_3216Metric_Pad1.33x1.80mm_HandSolder")
+      (reference "C11") (unit 1) (value "4700p") (footprint "Capacitor_SMD:C_1812_4532Metric_Pad1.57x3.40mm_HandSolder")
     )
     (path "/6235df39-6fe4-4ff0-a6f7-da05e5c190f5"
-      (reference "C12") (unit 1) (value "4700p") (footprint "Capacitor_SMD:C_1206_3216Metric_Pad1.33x1.80mm_HandSolder")
+      (reference "C12") (unit 1) (value "4700p") (footprint "Capacitor_SMD:C_1812_4532Metric_Pad1.57x3.40mm_HandSolder")
     )
     (path "/efe23ee3-88d7-4a07-85ed-8af6a1b1b716"
@@
       (reference "J3") (unit 1) (value "1-406541-1") (footprint "MJ406541:1-406541-1")
     )
-    (path "/bfa46546-c392-46f2-9dd1-54c070a9f47d"
-      (reference "L1") (unit 1) (value "PM6C-2004F") (footprint "PM6C-200XF:PM6C-2004F_SOP48")
-    )
     (path "/98624091-3add-4002-a75e-32916797ae00"
       (reference "R1") (unit 1) (value "75") (footprint "Resistor_SMD:R_0805_2012Metric_Pad1.20x1.40mm_HandSolder")
@@
       (reference "R8") (unit 1) (value "75") (footprint "Resistor_SMD:R_0805_2012Metric_Pad1.20x1.40mm_HandSolder")
     )
-  )
+    (path "/bfa46546-c392-46f2-9dd1-54c070a9f47d"
+      (reference "T1") (unit 1) (value "PM6C-2004F") (footprint "PM6C-200XF:PM6C-2004F_SOP48")
+    )
+  )

Commit message: update
Parts:
- C10, C9: value 1000p -> 1n
- C11, C12: value 4700p -> 4.7n
- renumbered R4 to R1, R3 to R2, R2 to R3, R1 to R4, R8 to R5, R7 to R6, R6 to R7, R5 to R8
Changed lines of the file:
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@@
   (symbol (lib_id "Device:R") (at 173.99 115.57 0) (unit 1)
     (in_bom yes) (on_board yes)
-    (property "Reference" "R7" (id 0) (at 172.72 114.3 0)
+    (property "Reference" "R6" (id 0) (at 172.72 114.3 0)
       (effects (font (size 1.27 1.27)) (justify left))
     )
@@
   (symbol (lib_id "Device:R") (at 171.45 85.09 0) (unit 1)
     (in_bom yes) (on_board yes)
-    (property "Reference" "R2" (id 0) (at 170.18 83.82 0)
+    (property "Reference" "R3" (id 0) (at 170.18 83.82 0)
       (effects (font (size 1.27 1.27)) (justify left))
     )
@@
   (symbol (lib_id "Device:R") (at 176.53 115.57 0) (unit 1)
     (in_bom yes) (on_board yes)
-    (property "Reference" "R8" (id 0) (at 175.26 114.3 0)
+    (property "Reference" "R5" (id 0) (at 175.26 114.3 0)
       (effects (font (size 1.27 1.27)) (justify left))
     )
@@
   (symbol (lib_id "Device:R") (at 171.45 115.57 0) (unit 1)
     (in_bom yes) (on_board yes)
-    (property "Reference" "R6" (id 0) (at 170.18 114.3 0)
+    (property "Reference" "R7" (id 0) (at 170.18 114.3 0)
       (effects (font (size 1.27 1.27)) (justify left))
     )
@@
       (effects (font (size 1.27 1.27)) (justify left))
     )
-    (property "Value" "4700p" (id 1) (at 149.86 138.43 90)
+    (property "Value" "4.7n" (id 1) (at 149.86 138.43 90)
       (effects (font (size 1.27 1.27)) (justify left))
     )
@@
   (symbol (lib_id "Device:R") (at 168.91 115.57 0) (unit 1)
     (in_bom yes) (on_board yes)
-    (property "Reference" "R5" (id 0) (at 167.64 114.3 0)
+    (property "Reference" "R8" (id 0) (at 167.64 114.3 0)
       (effects (font (size 1.27 1.27)) (justify left))
     )
@@
   (symbol (lib_id "Device:R") (at 176.53 85.09 0) (unit 1)
     (in_bom yes) (on_board yes)
-    (property "Reference" "R4" (id 0) (at 175.26 83.82 0)
+    (property "Reference" "R1" (id 0) (at 175.26 83.82 0)
       (effects (font (size 1.27 1.27)) (justify left))
     )
@@
       (effects (font (size 1.27 1.27)) (justify left))
     )
-    (property "Value" "1000p" (id 1) (at 189.23 119.38 90)
+    (property "Value" "1n" (id 1) (at 189.23 119.38 90)
       (effects (font (size 1.27 1.27)) (justify left))
     )
@@
       (effects (font (size 1.27 1.27)) (justify left))
     )
-    (property "Value" "4700p" (id 1) (at 149.86 133.35 90)
+    (property "Value" "4.7n" (id 1) (at 149.86 133.35 90)
       (effects (font (size 1.27 1.27)) (justify left))
     )
@@
   (symbol (lib_id "Device:R") (at 168.91 85.09 0) (unit 1)
     (in_bom yes) (on_board yes)
-    (property "Reference" "R1" (id 0) (at 167.64 83.82 0)
+    (property "Reference" "R4" (id 0) (at 167.64 83.82 0)
       (effects (font (size 1.27 1.27)) (justify left))
     )
@@
       (effects (font (size 1.27 1.27)) (justify left))
     )
-    (property "Value" "1000p" (id 1) (at 189.23 87.63 90)
+    (property "Value" "1n" (id 1) (at 189.23 87.63 90)
       (effects (font (size 1.27 1.27)) (justify left))
     )
@@
   (symbol (lib_id "Device:R") (at 173.99 85.09 0) (unit 1)
     (in_bom yes) (on_board yes)
-    (property "Reference" "R3" (id 0) (at 172.72 83.82 0)
+    (property "Reference" "R2" (id 0) (at 172.72 83.82 0)
       (effects (font (size 1.27 1.27)) (justify left))
     )
@@
     )
     (path "/b359cff7-6ac7-45fb-b749-9bcb9a702089"
-      (reference "C9") (unit 1) (value "1000p") (footprint "Capacitor_SMD:C_0805_2012Metric_Pad1.18x1.45mm_HandSolder")
+      (reference "C9") (unit 1) (value "1n") (footprint "Capacitor_SMD:C_0805_2012Metric_Pad1.18x1.45mm_HandSolder")
     )
     (path "/8b687076-a1d3-4ddc-b349-bb354de157f8"
-      (reference "C10") (unit 1) (value "1000p") (footprint "Capacitor_SMD:C_0805_2012Metric_Pad1.18x1.45mm_HandSolder")
+      (reference "C10") (unit 1) (value "1n") (footprint "Capacitor_SMD:C_0805_2012Metric_Pad1.18x1.45mm_HandSolder")
     )
     (path "/8fadaaf1-6657-4bb6-bf18-fe2c1d6327ef"
-      (reference "C11") (unit 1) (value "4700p") (footprint "Capacitor_SMD:C_1812_4532Metric_Pad1.57x3.40mm_HandSolder")
+      (reference "C11") (unit 1) (value "4.7n") (footprint "Capacitor_SMD:C_1812_4532Metric_Pad1.57x3.40mm_HandSolder")
     )
     (path "/6235df39-6fe4-4ff0-a6f7-da05e5c190f5"
-      (reference "C12") (unit 1) (value "4700p") (footprint "Capacitor_SMD:C_1812_4532Metric_Pad1.57x3.40mm_HandSolder")
+      (reference "C12") (unit 1) (value "4.7n") (footprint "Capacitor_SMD:C_1812_4532Metric_Pad1.57x3.40mm_HandSolder")
     )
     (path "/efe23ee3-88d7-4a07-85ed-8af6a1b1b716"
@@
       (reference "J3") (unit 1) (value "1-406541-1") (footprint "MJ406541:1-406541-1")
     )
+    (path "/8800c0ea-e18d-4861-805f-0285d3af2a43"
+      (reference "R1") (unit 1) (value "75") (footprint "Resistor_SMD:R_0805_2012Metric_Pad1.20x1.40mm_HandSolder")
+    )
+    (path "/b56d9773-4ef7-400f-a630-c6c1e23eaa14"
+      (reference "R2") (unit 1) (value "75") (footprint "Resistor_SMD:R_0805_2012Metric_Pad1.20x1.40mm_HandSolder")
+    )
+    (path "/214be8b9-04fb-43c8-a8e0-047e771dec58"
+      (reference "R3") (unit 1) (value "75") (footprint "Resistor_SMD:R_0805_2012Metric_Pad1.20x1.40mm_HandSolder")
+    )
     (path "/98624091-3add-4002-a75e-32916797ae00"
-      (reference "R1") (unit 1) (value "75") (footprint "Resistor_SMD:R_0805_2012Metric_Pad1.20x1.40mm_HandSolder")
-    )
-    (path "/214be8b9-04fb-43c8-a8e0-047e771dec58"
-      (reference "R2") (unit 1) (value "75") (footprint "Resistor_SMD:R_0805_2012Metric_Pad1.20x1.40mm_HandSolder")
-    )
-    (path "/b56d9773-4ef7-400f-a630-c6c1e23eaa14"
-      (reference "R3") (unit 1) (value "75") (footprint "Resistor_SMD:R_0805_2012Metric_Pad1.20x1.40mm_HandSolder")
-    )
-    (path "/8800c0ea-e18d-4861-805f-0285d3af2a43"
       (reference "R4") (unit 1) (value "75") (footprint "Resistor_SMD:R_0805_2012Metric_Pad1.20x1.40mm_HandSolder")
     )
+    (path "/24b50098-aeac-4460-91e0-b7c4b60de347"
+      (reference "R5") (unit 1) (value "75") (footprint "Resistor_SMD:R_0805_2012Metric_Pad1.20x1.40mm_HandSolder")
+    )
+    (path "/0d750a2c-84a4-469f-b267-be499eae4797"
+      (reference "R6") (unit 1) (value "75") (footprint "Resistor_SMD:R_0805_2012Metric_Pad1.20x1.40mm_HandSolder")
+    )
+    (path "/3021478b-fcd0-43c4-8f68-f5bf83e0352c"
+      (reference "R7") (unit 1) (value "75") (footprint "Resistor_SMD:R_0805_2012Metric_Pad1.20x1.40mm_HandSolder")
+    )
     (path "/7cb5ac04-2232-4d88-ac55-aab01928ac7c"
-      (reference "R5") (unit 1) (value "75") (footprint "Resistor_SMD:R_0805_2012Metric_Pad1.20x1.40mm_HandSolder")
-    )
-    (path "/3021478b-fcd0-43c4-8f68-f5bf83e0352c"
-      (reference "R6") (unit 1) (value "75") (footprint "Resistor_SMD:R_0805_2012Metric_Pad1.20x1.40mm_HandSolder")
-    )
-    (path "/0d750a2c-84a4-469f-b267-be499eae4797"
-      (reference "R7") (unit 1) (value "75") (footprint "Resistor_SMD:R_0805_2012Metric_Pad1.20x1.40mm_HandSolder")
-    )
-    (path "/24b50098-aeac-4460-91e0-b7c4b60de347"
       (reference "R8") (unit 1) (value "75") (footprint "Resistor_SMD:R_0805_2012Metric_Pad1.20x1.40mm_HandSolder")
     )
